File: nightstand-wifi-controller-pcb/nightstand-wifi-controller-pcb.kicad_pcb (KiCad board)
At the start: 2 copper layers, 67.4 x 54.8 mm, 11 parts, among them J1 Conn_01x02_Socket, J2 Conn_01x06_Socket, J4 Screw_Terminal_01x02, J5 Screw_Terminal_01x02, K2 FINDER-36.11, Q2 PN2222A

Commit message: Fix on earth for mcu module
Connections:
- LUATOS_ESP32C1 pad 32: unconnected-(LUATOS_ESP32C1-GND-Pad32) -> GND
Changed lines of the file:
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@@
   (net 37 "unconnected-(LUATOS_ESP32C1-GPIO08-Pad29)")
   (net 38 "unconnected-(LUATOS_ESP32C1-5V-Pad31)")
-  (net 39 "unconnected-(LUATOS_ESP32C1-GND-Pad32)")
   (footprint "TerminalBlock:TerminalBlock_Altech_AK300-2_P5.00mm" (layer "F.Cu")
     (at 91.195 68.82 180)
@@
       (net 38 "unconnected-(LUATOS_ESP32C1-5V-Pad31)") (pinfunction "5V") (pintype "power_out+no_connect"))
     (pad "32" thru_hole circle (at 19.3885 44.55) (size 1.524 1.524) (drill 0.762) (layers "*.Cu" "*.Mask")
-      (net 39 "unconnected-(LUATOS_ESP32C1-GND-Pad32)") (pinfunction "GND") (pintype "power_in"))
+      (net 35 "GND") (pinfunction "GND") (pintype "power_in"))
     (pad "32" smd rect (at 19.3885 44.55) (size 3.175 1.524) (drill (offset 0.9 0)) (layers "F.Cu" "F.Mask")
-      (net 39 "unconnected-(LUATOS_ESP32C1-GND-Pad32)") (pinfunction "GND") (pintype "power_in"))
+      (net 35 "GND") (pinfunction "GND") (pintype "power_in"))
   )
   (footprint "Relay_THT:Relay_SPDT_Finder_36.11" (layer "F.Cu")

Commit message: Snubber diod added to relay coil and temp sensor socket location fixed
Parts:
- added D1: 1N4001, Diode_THT:D_DO-41_SOD81_P10.16mm_Horizontal, F.Cu at (114.7, 84.9)
- moved J2 13.4 mm to (145.8, 101.4), turned to 180 degrees
- moved Q2 2.15 mm to (105.2, 88.5)
Routing:
- net Net-(J2-Pin_1): track 8.39 -> 32.6 mm
- net Net-(D1-K): track 57.2 -> 66.6 mm
- net Net-(D1-A): track 9.21 -> 15.9 mm
- net Net-(Q2-B): track 8.52 -> 12.6 mm
